File: kicad/nb1ecu.kicad_pcb (KiCad board)
At the start: 4 copper layers, 154 x 159 mm, 126 parts, among them J1 Conn_01x01, J1 Conn_02x03_Top_Bottom, J2 Conn_01x01, J2 Conn_01x02, J3 Conn_01x01, J4 Conn_01x01, J5 Conn_01x01, J6 Conn_01x01, P2 178780-1, Q1 PN2907A, Q10 DMG2302U, Q11 DMG2302U, Q12 DMG2302U, Q13 DMG2302U, Q14 DMG2302U, Q15 DMG2302U, Q16 DMG2302U, Q17 DMG2302U, Q2 PN2907A, Q3 DMG2302U, Q4 DMG2302U, Q5 DMG2302U, Q6 DMG2305UX, Q8 DMG2302U, Q9 DMG2302U, U1 Teensy4.1, U13 LMV324LIDT, U2 TL431LP, U3 MPX4250, U4 TC4424AVOA, U5 AP63205WU, U6 TC4424AVOA, U8 MPXHZ6115A, U9 SN65HVD232

Commit message: Official V1.0 milestone, all parts ordered
Parts:
- added J3: AudioPlug3, Connector_Audio:Jack_3.5mm_CUI_SJ1-3525N_Horizontal, F.Cu at (160.6, 120.2)
- added J4: Conn_01x03_Pin, Connector_PinSocket_2.54mm:PinSocket_1x03_P2.54mm_Vertical, F.Cu at (93.1, 63.1)
Connections:
- U4 pad 6: +5V -> Net-(J4-Pin_2)
- U6 pad 6: +5V -> Net-(J4-Pin_2)
Routing:
- net /KNOCK_SENS: track 0.00 -> 195.3 mm
- net Net-(J4-Pin_2): track 0.00 -> 44.9 mm, vias 0 -> 4
- net +5V: track 277.5 -> 236.1 mm, vias 3 -> 0
- net /O2_IA: track 50.0 -> 68.6 mm
- net /O2_VM: track 61.6 -> 51.8 mm, vias 0 -> 1
- net /O2_HEAT+: track 61.4 -> 69.1 mm
- net /O2_HEAT-: track 68.3 -> 60.7 mm
- net GND: track 209.2 -> 215.1 mm, vias 55 -> 59
- net /12V_IGN: track 348.4 -> 352.5 mm
- net /O2_IP: track 61.6 -> 65.4 mm, vias 0 -> 1
- net /O2_UN: track 63.0 -> 61.4 mm, vias 0 -> 1
Other:
- board text added: "12V"
- board text added: "5V"
- board text added: "Docs and config at: https://github.com/swagprincess/ecudocumentation"
- board text added: "IGN V"
- board text removed: "Docs and basemaps at: https://github.com/swagprincess/ecudocumentation"
