File: kicad/nb1ecu.kicad_sch (KiCad schematic)
At the start: 89 parts, among them P2 178780-1, Q1 PN2907A, Q10 DMG2302U, Q11 DMG2302U, Q12 DMG2302U, Q13 DMG2302U, Q14 DMG2302U, Q15 DMG2302U, Q16 DMG2302U, Q2 PN2907A, Q3 DMG2302U, Q4 DMG2302U, Q5 DMG2302U, Q6 DMG2305UX, Q7 DMG2305UX, Q8 DMG2302U, Q9 DMG2302U, U1 Teensy4.1, U13 LMV324LIDT, U2 TL431LP, U3 MPX4_MAP, U4 TC4424AVOA, U5 AP63205WU, U6 TC4424AVOA

Commit message: bunch of new features
Parts:
- removed Q7: DMG2305UX, Package_TO_SOT_SMD:SOT-23, symbol Transistor_FET:Q_PMOS_GSD
- added C10, C9: 220n, Capacitor_SMD:C_0805_2012Metric_Pad1.18x1.45mm_HandSolder, symbol Device:C
- added C20, C8: 100n, Capacitor_SMD:C_0805_2012Metric_Pad1.18x1.45mm_HandSolder, symbol Device:C
- added C21: 22n, Capacitor_SMD:C_0805_2012Metric_Pad1.18x1.45mm_HandSolder, symbol Device:C
- added Q17: DMG2302U, Package_TO_SOT_SMD:SOT-23, symbol Transistor_FET:DMG2302U
- added R47: 180k, Resistor_SMD:R_0805_2012Metric_Pad1.20x1.40mm_HandSolder, symbol Device:R_US
- added R48: 3.9k, Resistor_SMD:R_0805_2012Metric_Pad1.20x1.40mm_HandSolder, symbol Device:R_US
- added R49: 604, Resistor_SMD:R_0805_2012Metric_Pad1.20x1.40mm_HandSolder, symbol Device:R_US
- added R50: 470, Resistor_SMD:R_0805_2012Metric_Pad1.20x1.40mm_HandSolder, symbol Device:R_US
- added R51: 1k, Resistor_SMD:R_0805_2012Metric_Pad1.20x1.40mm_HandSolder, symbol Device:R_US
- added U8: MPXHZ6115A, Package_SO:SSOP-8_3.95x5.21x3.27mm_P1.27mm, symbol Sensor_Pressure:MPXHZ6115A
- C11: LCSC Part # C77069 -> C520079
- C12, C14, C16, C17: LCSC Part # C77069 -> C541527
- C13, C15, C18, C19, C5: LCSC Part # C1791 -> C520083
- L1: LCSC Part # (none) -> C82314
- LAMBDA_OUT1, U1: now left out of the parts list
- Q10, Q11, Q12, Q13, Q14, Q15, Q16, Q3, Q4, Q5, Q8, Q9: LCSC Part # (none) -> C96613
- Q6: LCSC Part # (none) -> C150470
- R11, R12, R14, R33, R34, R35, R45: LCSC Part # C865519 -> C855098
- R13: value 10k -> 48.7k
- R15, R16, R17, R18, R20, R21, R23, R25, R27, R38, R39, R40, R43, R44, R46: LCSC Part # C865519 -> C865232
- R19, R31: LCSC Part # C865519 -> C114564
- R22, R24, R26, R28: LCSC Part # C865519 -> C228757
- R29, R30: LCSC Part # C865519 -> C375522
- R41, R42: LCSC Part # C865519 -> C114519
- R8: LCSC Part # C3565480 -> C855098
- U2: LCSC Part # (none) -> C398376
- U3: value MPX4_MAP -> MPX4250; now left out of the parts list
Connections:
- net +3V3: now also C20.2, R51.2, U8.2 (Vcc)
- net +5V: no longer R13.1
- net 12V_IGN: now also R48.2
- net GND: now also R13.2, C10.2, C20.1, C21.1, C8.2, C9.2, Q17.2 (S), R47.1, R49.1, U8.3 (GND)
- net MAIN_FAN: now also U1.17 (25_A11_RX6_SDA2), Q17.1 (G), R47.2; no longer P2.20 (1R)
- net AC_OUT: now reaches Q8.1 (G), R45.2
- net AC_OUT: now also U1.22 (30_CRX3)
- net AC: now reaches U1.23 (31_CTX3)
- net AC: now also P2.19 (1P), C10.1, R51.1
- net BATT: now reaches U1.31 (39_MISO1_OUT1A)
- net BATT: now also C9.1, R50.1
- net BARO: now reaches U1.40 (18_A4_SDA)
- net BARO: now also R13.1, C21.2, U8.4 (Vout)
- removed net AC_SWITCH: P2.19 (1P), R13.2
- new net: C8.1, R48.1, R49.2, R50.2
- new net MAIN_FAN_OUT: P2.20 (1R), Q17.3 (D)
Other:
- note added: "AC SWITCH"
- note added: "BARO"
- note added: "BATTERY"
- note added: "FAN"
- moved on the sheet: C17, Q8, R32, R45

Commit message: options connector
Parts:
- removed LAMBDA_OUT1: TestPoint, TestPoint:TestPoint_Pad_3.0x3.0mm, symbol Connector:TestPoint
- added C22: 220n, Capacitor_SMD:C_0805_2012Metric_Pad1.18x1.45mm_HandSolder, symbol Device:C
- added J1: Conn_02x03_Top_Bottom, Connector_Molex:Molex_Micro-Fit_3.0_43045-0600_2x03_P3.00mm_Horizontal, symbol Connector_Generic:Conn_02x03_Top_Bottom
- added R52: 1k, Resistor_SMD:R_0805_2012Metric_Pad1.20x1.40mm_HandSolder, symbol Device:R_US
Connections:
- net +3V3: now also R52.2
- net +5V: now also J1.3 (Pin_3)
- net 12V_IGN: now also J1.2 (Pin_2)
- net GND: now also C22.2, J1.1 (Pin_1)
- net LAMBDA_5V: now also J1.4 (Pin_4)
- net VICS_OUT: now also J1.5 (Pin_5)
- net SPARE_DIGITAL_1: now reaches U1.24 (32_OUT1B)
- net SPARE_DIGITAL_1: now also C22.1, J1.6 (Pin_6), R52.1
Other:
- note added: "AUX1DIGITAL"
- moved on the sheet: Q4, R34

Commit message: add CANBUS
Parts:
- added C23: 220n, Capacitor_SMD:C_0805_2012Metric_Pad1.18x1.45mm_HandSolder, symbol Device:C
- added D1, D10, D2, D3, D4, D5, D6, D7, D8, D9: SMF15A, Diode_SMD:D_SMF, symbol Diode:SMF15A
- added J2: Conn_01x02, Connector_Molex:Molex_Micro-Fit_3.0_43650-0200_1x02_P3.00mm_Horizontal, symbol Connector_Generic:Conn_01x02
- added JP1: SolderJumper_2_Open, Jumper:SolderJumper-2_P1.3mm_Open_Pad1.0x1.5mm, symbol Jumper:SolderJumper_2_Open
- added R53: 1k, Resistor_SMD:R_0805_2012Metric_Pad1.20x1.40mm_HandSolder, symbol Device:R_US
- added R54: 120, Resistor_SMD:R_0805_2012Metric_Pad1.20x1.40mm_HandSolder, symbol Device:R_US
- added U9: SN65HVD232, Package_SO:SOIC-8_3.9x4.9mm_P1.27mm, symbol Interface_CAN_LIN:SN65HVD232
Connections:
- net +3V3: now also R53.2, U9.3 (VCC)
- net AC_FAN: now also D6.1 (A1)
- net BOOST_OUT: now also D9.1 (A1)
- net GND: now also C23.2, D1.2 (A2), D10.2 (A2), D2.2 (A2), D3.2 (A2), D4.2 (A2), D5.2 (A2), D6.2 (A2), D7.2 (A2), D8.2 (A2), D9.2 (A2), U9.2 (GND)
- net IAC_OUT: now also D5.1 (A1)
- net INJ1_OUT: now also D1.1 (A1)
- net INJ2_OUT: now also D2.1 (A1)
- net INJ3_OUT: now also D4.1 (A1)
- net INJ4_OUT: now also D3.1 (A1)
- net MAIN_FAN_OUT: now also D10.1 (A1)
- net PUMP_OUT: now also D8.1 (A1)
- net VICS_OUT: now also D7.1 (A1)
- net VSS_IN: now reaches P2.32 (2D)
- net VSS_IN: now also JP1.1 (A)
- net VSS: now reaches U1.33 (41_A17)
- net VSS: now also C23.1, JP1.2 (B), R53.1
- net CANTX: now reaches U1.44 (22_A8_CTX1)
- net CANTX: now also U9.1 (D)
- net CANRX: now reaches U1.45 (23_A9_CRX1_MCLK1)
- net CANRX: now also U9.4 (R)
- new net CANH: J2.1 (Pin_1), R54.1, U9.7 (CANH)
- new net CANL: J2.2 (Pin_2), R54.2, U9.6 (CANL)
Other:
- note added: "CAN"
- note added: "OPTION PORT 1"
- note added: "OPTION PORT 2"
- note added: "VSS"
- note added: "WIDEBAND SPARTAN 3 LITE OEM"
- note added: "molex microfit"
- note added: "options port counterpart numbers: 178845-6 917975-6"
- note removed: "WIDEBAND SPARTAN 3"
- note removed: "options port part numbers: 178845-6 917975-6"
- moved on the sheet: J1, U1

Commit message: revision
Parts:
- removed D1, D10, D2, D3, D4, D5, D6, D7, D8, D9: SMF15A, Diode_SMD:D_SMF, symbol Diode:SMF15A
- added D1, D10, D11, D2, D3, D4, D5, D6, D7, D8, D9: 1N4448W, Diode_SMD:D_SOD-123, symbol Diode:1N4448W
- added R55: 10k, Resistor_SMD:R_0805_2012Metric_Pad1.20x1.40mm_HandSolder, symbol Device:R_US
Connections:
- net +3V3: now also D11.1 (K), R55.1; no longer R53.2
- net 12V_IGN: now also D1.1 (K), D10.1 (K), D2.1 (K), D3.1 (K), D4.1 (K), D5.1 (K), D6.1 (K), D7.1 (K), D8.1 (K), D9.1 (K)
- net AC_FAN: now also D6.2 (A)
- net BOOST_OUT: now also D9.2 (A)
- net IAC_OUT: now also D5.2 (A)
- net INJ1_OUT: now also D1.2 (A)
- net INJ2_OUT: now also D2.2 (A)
- net INJ3: now also U1.11 (9_OUT1C); no longer U1.10 (8_TX2_IN1)
- net INJ3_OUT: now also D4.2 (A)
- net INJ4: now also U1.10 (8_TX2_IN1); no longer U1.11 (9_OUT1C)
- net INJ4_OUT: now also D3.2 (A)
- net MAIN_FAN_OUT: now also D10.2 (A)
- net PUMP_OUT: now also D8.2 (A)
- net VICS_OUT: now also D7.2 (A)
- net VSS: now also R53.2, D11.2 (A), R55.2; no longer JP1.2 (B), R53.1
- new net: JP1.2 (B), R53.1
Other:
- moved on the sheet: JP1, Q11, Q12, Q16, R39, R40, R46, R53

Commit message: Official V1.0 milestone, all parts ordered
Parts:
- added J3: AudioPlug3, Connector_Audio:Jack_3.5mm_CUI_SJ1-3525N_Horizontal, symbol Connector_Audio:AudioPlug3
- added J4: Conn_01x03_Pin, Connector_PinSocket_2.54mm:PinSocket_1x03_P2.54mm_Vertical, symbol Connector:Conn_01x03_Pin
- Q1, Q2: LCSC Part # C513106 -> C903222
Connections:
- net +5V: now also J4.1 (Pin_1); no longer U4.6 (VDD), U6.6 (VDD)
- net 12V_IGN: now also J4.3 (Pin_3)
- net GND: now also J3.S
- net KNOCK_SENS: now also J3.R, J3.T
- new net: J4.2 (Pin_2), U4.6 (VDD), U6.6 (VDD)
Other:
- moved on the sheet: R15, R16, R17, R18, U4, U6
